File: LaunchOps/FillControl/Schematic/FillControl/FillControl.sch (EAGLE design)
At the start: 48 parts

Commit message: transferring to PC
Parts:
- added C3, C4, C5, C6: (no value), rcl:C-EUC0402
- added D8, D9: (no value), FillControl:DIODE
- added F1: FUSE, FillControl:FUSE
- added K7, K8: (no value), FillControl:RELAY
- added R19, R20, R21, R22, R23, R24, R25, R26, R27, R28: (no value), rcl:R-US_R0603
- added U14, U15, U16, U17: (no value), FillControl:ADS1115IDGSR
- added U18, U20: (no value), FillControl:OPTOISOLATOR
- added U19, U21: (no value), FillControl:NPN_BJT
Connections:
- new net +24V: F1.1
- new net AIN1_A: U14.AIN0
- new net AIN1_B: U14.AIN1
- new net AIN2_A: U14.AIN3
- new net AIN2_B: U14.AIN2
- new net AIN3_A: U15.AIN0
- new net AIN3_B: U15.AIN1
- new net AIN4_A: U15.AIN3
- new net AIN4_B: U15.AIN2
- new net AIN5_A: U16.AIN0
- new net AIN5_B: U16.AIN1
- new net AIN6_A: U16.AIN3
- new net AIN6_B: U16.AIN2
- new net AIN7_A: U17.AIN0
- new net AIN7_B: U17.AIN1
- new net AIN8_A: U17.AIN3
- new net AIN8_B: U17.AIN2
- new net N$39: D8.2, K7.4, R22.2
- new net N$41: R23.1, U18.3
- new net N$42: R19.1, U14.ADDR
- new net N$43: R23.2, U19.B
- new net N$44: R22.1, U19.C
- new net N$45: R24.2, U18.2
- new net N$46: U18.1
- new net N$47: D9.2, K8.4, R25.2
- new net N$48: R26.1, U20.3
- new net N$49: R26.2, U21.B
- new net N$50: R25.1, U21.C
- new net N$51: R27.2, U20.2
- new net N$52: U20.1
- new net N$53: R28.1, U15.ADDR
- new net N$54: U17.ALERT/RDY
- new net N$55: U16.ALERT/RDY
- new net N$56: R19.2
- new net N$57: U15.ALERT/RDY
- new net N$58: U14.ALERT/RDY
- new net SCL: R21.1, U14.SCL, U15.SCL, U16.SCL, U17.ADDR, U17.SCL
- new net SDA: R20.1, U14.SDA, U15.SDA, U16.ADDR, U16.SDA, U17.SDA
- net +5V: now also C3.1, C4.1, C5.1, C6.1, D8.1, D9.1, K7.3, K8.3, R20.2, R21.2, R28.2, U14.VDD, U15.VDD, U16.VDD, U17.VDD, U18.4, U20.4
- net GND: now also C3.2, C4.2, C5.2, C6.2, R24.1, R27.1, U14.GND, U15.GND, U16.GND, U17.GND, U19.E, U21.E
- net N$40: now also F1.2
Other:
- moved on the sheet: C1, C2, D1, D2, D3, D4, D5, D6, D7, K1, K2, K3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

Commit message: Push cad to pc
Parts:
- removed D2, D3, D4, D5, D6, D8, D9: (no value), FillControl:DIODE
- removed K2, K3, K4, K5, K6, K7, K8: (no value), FillControl:RELAY
- removed R10, R11, R12, R13, R14, R15, R16, R17, R18, R22, R23, R24, R25, R26, R27, R4, R5, R6, R7, R8, R9: (no value), rcl:R-US_R0603
- removed U10, U12, U19, U21, U4, U6, U8: (no value), FillControl:NPN_BJT
- removed U11, U18, U20, U3, U5, U7, U9: (no value), FillControl:OPTOISOLATOR
- added J1: (no value), MICROCONTROLLER:20POS
- added J2: (no value), MICROCONTROLLER:16POS_CONN
- added R35, R36, R37, R38, R39, R40, R41, R42: (no value), rcl:R-US_R0603
Connections:
- removed net N$15: R8.2, U6.B
- removed net N$19: D4.2, K4.4, R10.2
- removed net N$20: R11.1, U7.3
- removed net N$21: R11.2, U8.B
- removed net N$22: R10.1, U8.C
- removed net N$23: R12.2, U7.2
- removed net N$24: U7.1
- removed net N$25: D5.2, K5.4, R13.2
- removed net N$26: R14.1, U9.3
- removed net N$27: R14.2, U10.B
- removed net N$28: R13.1, U10.C
- removed net N$29: R15.2, U9.2
- removed net N$30: U9.1
- removed net N$31: D6.2, K6.4, R16.2
- removed net N$32: R17.1, U11.3
- removed net N$33: R17.2, U12.B
- removed net N$34: R16.1, U12.C
- removed net N$35: R18.2, U11.2
- removed net N$36: U11.1
- removed net N$39: D8.2, K7.4, R22.2
- removed net N$41: R23.1, U18.3
- removed net N$43: R23.2, U19.B
- removed net N$44: R22.1, U19.C
- removed net N$45: R24.2, U18.2
- removed net N$46: U18.1
- removed net N$47: D9.2, K8.4, R25.2
- removed net N$48: R26.1, U20.3
- removed net N$49: R26.2, U21.B
- removed net N$50: R25.1, U21.C
- removed net N$51: R27.2, U20.2
- removed net N$52: U20.1
- new net N$71: J2.A1+, R35.2
- new net R1+: K1.5
- net +24V: now also K1.1
- net +5V: no longer D2.1, D3.1, D4.1, D5.1, D6.1, D8.1, D9.1, K2.3, K3.3, K4.3, K5.3, K6.3, K7.3, K8.3, U11.4, U18.4, U20.4, U3.4, U5.4, U7.4, U9.4
- net GND: no longer R12.1, R15.1, R18.1, R24.1, R27.1, R6.1, R9.1, U10.E, U12.E, U14.GND, U19.E, U21.E, U4.E, U6.E, U8.E
- net N$10: now also J2.A2-, R38.1; no longer R4.1, U4.C
- net N$11: now also R37.1, R38.2; no longer R6.2, U3.2
- net N$12: now also J2.A3-, R40.1; no longer U3.1
- net N$13: now also R39.1, R40.2; no longer D3.2, K3.4, R7.2
- net N$14: now also J2.A3+, R39.2; no longer R8.1, U5.3
- net N$16: now also R41.1, R42.2; no longer R7.1, U6.C
- net N$17: now also J2.A4+, R41.2; no longer R9.2, U5.2
- net N$18: now also J2.A4-, R42.1; no longer U5.1
- net N$56: now also U14.GND
- net N$7: now also J2.A1-, R36.1; no longer D2.2, K2.4, R4.2
- net N$8: now also R35.1, R36.2; no longer R5.1, U3.3
- net N$9: now also J2.A2+, R37.2; no longer R5.2, U4.B
Other:
- note added: "RELAY 1"
