File: LaunchOps/FillControl/Schematic/FillControl/FillControl.sch (EAGLE design)
At the start: 134 parts

Commit message: staging
Other:
- note added: "(-)"
- note added: "DESIGNED BY: J. BRANDON IAMS"
- note added: "INITIAL DEVELOPMENT"
Changed lines of the file:
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@@
 <setting verticaltext="up"/>
 </settings>
-<grid distance="0.1" unitdist="inch" unit="inch" style="dots" multiple="1" display="yes" altdistance="0.01" altunitdist="inch" altunit="inch"/>
+<grid distance="0.1" unitdist="inch" unit="inch" style="lines" multiple="1" display="no" altdistance="0.01" altunitdist="inch" altunit="inch"/>
 <layers>
 <layer number="1" name="Top" color="4" fill="1" visible="no" active="no"/>
@@
 <text x="124.46" y="142.24" size="3.81" layer="97">ADC1</text>
 <text x="124.46" y="86.36" size="3.81" layer="97">ADC2</text>
+<text x="338.074" y="6.604" size="3.81" layer="95">INITIAL DEVELOPMENT</text>
+<text x="417.322" y="6.096" size="3.81" layer="95">(-)</text>
+<text x="327.66" y="27.94" size="3.81" layer="96">DESIGNED BY: J. BRANDON IAMS</text>
 </plain>
 <instances>
@@
 <text x="287.02" y="93.98" size="3.81" layer="97" rot="R270">RELAY OUT</text>
 <text x="386.08" y="91.44" size="3.81" layer="97" rot="R270">LED OUT</text>
+<text x="338.074" y="6.604" size="3.81" layer="95">INITIAL DEVELOPMENT</text>
+<text x="417.322" y="6.096" size="3.81" layer="95">(-)</text>
+<text x="327.66" y="27.94" size="3.81" layer="96">DESIGNED BY: J. BRANDON IAMS</text>
 </plain>
 <instances>
