File: LaunchOps/FillControl/Schematic/FillControl/FillControl.brd (EAGLE design)
At the start: 200 x 200 mm, 134 parts

Commit message: staging
Parts:
- moved D2 309.2 mm to (162.8, 39.4), turned to 180 degrees
- moved D3 298.0 mm to (146.1, 39.0), turned to 180 degrees
- moved R6 281.6 mm to (157.3, 51.9)
- moved R4 280.1 mm to (156.6, 40.1), turned to 270 degrees
- moved R5 279.7 mm to (157.3, 48.8), turned to 180 degrees
- moved R9 276.1 mm to (139.7, 52.0)
- moved R7 275.4 mm to (139.6, 40.0), turned to 270 degrees
- moved R8 274.4 mm to (139.7, 48.6), turned to 180 degrees
- moved R10 268.2 mm to (122.4, 40.3), turned to 270 degrees
- moved U4 256.2 mm to (157.2, 44.3), turned to 270 degrees
- moved U6 245.2 mm to (139.6, 44.4), turned to 270 degrees
- moved U8 234.5 mm to (122.6, 45.5), turned to 270 degrees
- moved R11 227.3 mm to (122.5, 49.2), turned to 180 degrees
- moved U3 226.1 mm to (164.6, 48.0), turned to 270 degrees
- moved U10 224.9 mm to (105.6, 44.5), turned to 270 degrees
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Routing:
- net +5V: track 24.7 -> 235.2 mm
- net N$8: track 0.00 -> 26.7 mm
- net R7+: track 0.00 -> 11.8 mm
- net R2+: track 0.00 -> 11.8 mm
- net R6+: track 0.00 -> 11.8 mm
- net R5+: track 0.00 -> 11.8 mm
- net R4+: track 0.00 -> 11.8 mm
- net R10+: track 0.00 -> 11.8 mm
- net R9+: track 0.00 -> 11.8 mm
- net R3+: track 0.00 -> 11.8 mm
- net R8+: track 0.00 -> 11.4 mm
- net N$27: track 0.00 -> 10.4 mm
- net N$21: track 0.00 -> 10.3 mm
- net N$72: track 0.00 -> 10.2 mm
- net N$43: track 0.00 -> 9.86 mm
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