File: DevelopmentMCU/dev_A.sch (EAGLE design)
At the start: 3 parts, among them U1 TM4C123_DEVICE, U2 AP2112K-3.3TRG1

Commit message: Library almost finished
Parts:
- removed U2: AP2112K-3.3TRG1, AP2112K-3.3TRG1:AP2112K-3.3TRG1
- added U$2, U$3: (no value), MICROCONTROLLER:SWITCH_B3S
- added U$4: (no value), MICROCONTROLLER:RGBLED
- U$1: value MCP73831T-2ATI/OT -> (none); device MICROCONTROLLER:MCP73831T-2ATI/OT -> MICROCONTROLLER:SWITCH_B3S
Other:
- moved on the sheet: U1
Changed lines of the file:
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@@
 <layers>
 <layer number="1" name="Top" color="4" fill="1" visible="no" active="no"/>
-<layer number="2" name="Route2" color="16" fill="1" visible="no" active="no"/>
-<layer number="3" name="Route3" color="17" fill="1" visible="no" active="no"/>
-<layer number="4" name="Route4" color="18" fill="1" visible="no" active="no"/>
-<layer number="5" name="Route5" color="19" fill="1" visible="no" active="no"/>
-<layer number="6" name="Route6" color="25" fill="1" visible="no" active="no"/>
-<layer number="7" name="Route7" color="26" fill="1" visible="no" active="no"/>
-<layer number="8" name="Route8" color="27" fill="1" visible="no" active="no"/>
-<layer number="9" name="Route9" color="28" fill="1" visible="no" active="no"/>
-<layer number="10" name="Route10" color="29" fill="1" visible="no" active="no"/>
-<layer number="11" name="Route11" color="30" fill="1" visible="no" active="no"/>
-<layer number="12" name="Route12" color="20" fill="1" visible="no" active="no"/>
-<layer number="13" name="Route13" color="21" fill="1" visible="no" active="no"/>
-<layer number="14" name="Route14" color="22" fill="1" visible="no" active="no"/>
-<layer number="15" name="Route15" color="23" fill="1" visible="no" active="no"/>
+<layer number="2" name="Route2" color="1" fill="3" visible="no" active="no"/>
+<layer number="3" name="Route3" color="4" fill="3" visible="no" active="no"/>
+<layer number="4" name="Route4" color="1" fill="4" visible="no" active="no"/>
+<layer number="5" name="Route5" color="4" fill="4" visible="no" active="no"/>
+<layer number="6" name="Route6" color="1" fill="8" visible="no" active="no"/>
+<layer number="7" name="Route7" color="4" fill="8" visible="no" active="no"/>
+<layer number="8" name="Route8" color="1" fill="2" visible="no" active="no"/>
+<layer number="9" name="Route9" color="4" fill="2" visible="no" active="no"/>
+<layer number="10" name="Route10" color="1" fill="7" visible="no" active="no"/>
+<layer number="11" name="Route11" color="4" fill="7" visible="no" active="no"/>
+<layer number="12" name="Route12" color="1" fill="5" visible="no" active="no"/>
+<layer number="13" name="Route13" color="4" fill="5" visible="no" active="no"/>
+<layer number="14" name="Route14" color="1" fill="6" visible="no" active="no"/>
+<layer number="15" name="Route15" color="4" fill="6" visible="no" active="no"/>
 <layer number="16" name="Bottom" color="1" fill="1" visible="no" active="no"/>
 <layer number="17" name="Pads" color="2" fill="1" visible="no" active="no"/>
 <layer number="18" name="Vias" color="2" fill="1" visible="no" active="no"/>
 <layer number="19" name="Unrouted" color="6" fill="1" visible="no" active="no"/>
-<layer number="20" name="Dimension" color="24" fill="1" visible="no" active="no"/>
+<layer number="20" name="Dimension" color="15" fill="1" visible="no" active="no"/>
 <layer number="21" name="tPlace" color="7" fill="1" visible="no" active="no"/>
 <layer number="22" name="bPlace" color="7" fill="1" visible="no" active="no"/>
@@
 <layer number="97" name="Info" color="7" fill="1" visible="yes" active="yes"/>
 <layer number="98" name="Guide" color="6" fill="1" visible="yes" active="yes"/>
+<layer number="99" name="SpiceOrder" color="7" fill="1" visible="yes" active="yes"/>
 </layers>
 <schematic xreflabel="%F%N/%S.%C%R" xrefpart="/%S.%C%R">
@@
 </classes>
 <parts>
+<part name="FRAME1" library="frames" library_urn="urn:adsk.eagle:library:229" deviceset="FRAME_B_L" device=""/>
 <part name="U1" library="MICROCONTROLLER" deviceset="TM4C123_DEVICE" device="" package3d_urn="urn:adsk.eagle:package:14363313/1"/>
-<part name="FRAME1" library="frames" library_urn="urn:adsk.eagle:library:229" deviceset="FRAME_B_L" device=""/>
-<part name="U2" library="AP2112K-3.3TRG1" deviceset="AP2112K-3.3TRG1" device=""/>
-<part name="U$1" library="MICROCONTROLLER" deviceset="MCP73831T-2ATI/OT" device="" package3d_urn="urn:adsk.eagle:package:14364640/1"/>
+<part name="U$1" library="MICROCONTROLLER" deviceset="SWITCH_B3S" device=""/>
+<part name="U$2" library="MICROCONTROLLER" deviceset="SWITCH_B3S" device=""/>
+<part name="U$3" library="MICROCONTROLLER" deviceset="SWITCH_B3S" device=""/>
+<part name="U$4" library="MICROCONTROLLER" deviceset="RGBLED" device=""/>
 </parts>
 <sheets>
@@
 </plain>
 <instances>
-<instance part="U1" gate="A" x="96.52" y="195.58" smashed="yes">
-<attribute name="NAME" x="129.8956" y="204.6986" size="2.0828" layer="95" ratio="6" rot="SR0"/>
-<attribute name="VALUE" x="129.2606" y="202.1586" size="2.0828" layer="96" ratio="6" rot="SR0"/>
-</instance>
 <instance part="FRAME1" gate="G$1" x="0" y="0" smashed="yes"/>
 <instance part="FRAME1" gate="G$2" x="325.12" y="0" smashed="yes">
@@
 <attribute name="DRAWING_NAME" x="342.9" y="19.05" size="2.54" layer="94"/>
 </instance>
-<instance part="U2" gate="G$1" x="198.12" y="231.14" smashed="yes">
-<attribute name="NAME" x="190.45705" y="239.787609375" size="2.08946875" layer="95" ratio="10" rot="SR0"/>
-<attribute name="VALUE" x="190.4711" y="219.4893" size="2.0883" layer="96" ratio="10" rot="SR0"/>
+<instance part="U1" gate="A" x="73.66" y="167.64" smashed="yes">
+<attribute name="NAME" x="107.0356" y="176.7586" size="2.0828" layer="95" ratio="6" rot="SR0"/>
+<attribute name="VALUE" x="106.4006" y="174.2186" size="2.0828" layer="96" ratio="6" rot="SR0"/>
 </instance>
-<instance part="U$1" gate="A" x="259.08" y="220.98" smashed="yes">
-<attribute name="NAME" x="251.46" y="241.3" size="1.27" layer="95"/>
-<attribute name="VALUE" x="251.46" y="226.06" size="1.27" layer="96"/>
+<instance part="U$1" gate="A" x="177.8" y="142.24" smashed="yes">
+<attribute name="NAME" x="174.752" y="147.066" size="1.778" layer="95"/>
+<attribute name="VALUE" x="173.99" y="136.652" size="1.778" layer="96"/>
 </instance>
+<instance part="U$2" gate="A" x="177.8" y="129.54" smashed="yes">
+<attribute name="NAME" x="174.752" y="134.366" size="1.778" layer="95"/>
+<attribute name="VALUE" x="173.99" y="123.952" size="1.778" layer="96"/>
+</instance>
+<instance part="U$3" gate="A" x="177.8" y="116.84" smashed="yes">
+<attribute name="NAME" x="174.752" y="121.666" size="1.778" layer="95"/>
+<attribute name="VALUE" x="173.99" y="111.252" size="1.778" layer="96"/>
+</instance>
+<instance part="U$4" gate="A" x="271.78" y="144.78" smashed="yes"/>
 </instances>
 <busses>

Commit message: second commit
Parts:
- removed U$3: (no value), MICROCONTROLLER:SWITCH_B3S
- added RESET, SW1, SW2: (no value), MICROCONTROLLER:SWITCH_B3S
- U$1: device MICROCONTROLLER:SWITCH_B3S -> MICROCONTROLLER:HEADER_J1
- U$2: device MICROCONTROLLER:SWITCH_B3S -> MICROCONTROLLER:HEADER_J2
Connections:
- new net N$1: U$1.PA2, U1.PA2/SSI0CLK
- new net N$10: U$1.PB3, U1.PB3/I2C0SDA
- new net N$11: U$1.PB4, U1.PB4
- new net N$12: U$1.PB5, U1.PB5
- new net N$13: U$1.PB6, U1.PB6
- new net N$14: U$1.PB7, U1.PB7
- new net N$15: U$1.PC4, U1.PC4
- new net N$16: U$1.PC5, U1.PC5
- new net N$17: U$1.PC6, U1.PC6
- new net N$18: U$1.PC7, U1.PC7
- new net N$19: U$2.PD0, U1.PD0
- new net N$2: U$1.PA3, U1.PA3/SSI0FSS
- new net N$20: U$2.PD1, U1.PD1
- new net N$21: U$2.PD2, U1.PD2
- new net N$22: U$2.PD3, U1.PD3
- new net N$23: U$2.PD6, U1.PD6
- new net N$24: U$2.PD7, U1.PD7
- new net N$25: U$2.PE0, U1.PE0
- new net N$26: U$2.PE1, U1.PE1
- new net N$27: U$2.PE2, U1.PE2
- new net N$28: U$2.PE3, U1.PE3
- new net N$29: U$2.PE4, U1.PE4
- new net N$3: U$1.PA4, U1.PA4/SSI0RX
- new net N$30: U$2.PE5, U1.PE5
- new net N$31: U$2.PF0, U1.PF0
- new net N$32: U$2.PF1, U1.PF1
- new net N$33: U$2.PF2, U1.PF2
- new net N$34: U$2.PF3, U1.PF3
- new net N$35: U$2.PF4, U1.PF4
- new net N$4: U$1.PA5, U1.PA5/SSI0TX
- new net N$5: U$1.PA6, U1.PA6
- new net N$6: U$1.PA7, U1.PA7
- new net N$7: U$1.PB0, U1.PB0/USB0ID
- new net N$8: U$1.PB1, U1.PB1/USB0VBUS
- new net N$9: U$1.PB2, U1.PB2/I2C0SCL
Other:
- moved on the sheet: U1

Commit message: Staging
Parts:
- added R1: 330, MICROCONTROLLER:RESISTOR
- added R28: 10k, MICROCONTROLLER:RESISTOR
Connections:
- net N$32 renamed LED_R
- net N$33 renamed LED_B
- net N$34 renamed LED_G
- removed net N$35: U$2.PF4, U1.PF4
- new net !WAKE: R1.1
- new net +MCU_PWR: R28.2
- new net GND: RESET.1@A, RESET.1@B, SW1.1@A, SW1.1@B, SW2.1@A, SW2.1@B
- new net RST: U$2.RST
- new net SW1: SW1.0@A, SW1.0@B, U$2.PF4, U1.PF4
- new net SW2: R1.2, SW2.0@A, SW2.0@B, U$2.PF0, U1.PF0
- net N$31: now also R28.1, RESET.0@A, RESET.0@B; no longer U$2.PF0, U1.PF0
Other:
- moved on the sheet: RESET, SW1, SW2, U$2

Commit message: Staging
Parts:
- removed R28: 10k, MICROCONTROLLER:RESISTOR
- added R2: 10k, MICROCONTROLLER:RESISTOR
- added R3, R4, R5: 330, MICROCONTROLLER:RESISTOR
- added U$3, U$5, U$6: (no value), MICROCONTROLLER:NPN_BJT
- added U$7: 32kHz, MICROCONTROLLER:32KHZ_OSCILATOR
- added U$8, U$9: (no value), MICROCONTROLLER:CAPACITOR
Connections:
- new net +VBUS: U$4.4
- new net N$32: R3.2, U$4.1
- new net N$33: R4.2, U$4.2
- new net N$34: R5.2, U$4.3
- new net N$35: R5.1, U$6.C
- new net N$36: R4.1, U$5.C
- new net N$37: R3.1, U$3.C
- new net N$38: U$7.2, U$8.1, U1.OSC0
- new net N$39: U$7.1, U$9.2, U1.OSC1
- new net N$40: U$8.2, U$9.1, U1.GNDX
- net +MCU_PWR: now also R2.2; no longer R28.2
- net GND: now also U$3.E, U$5.E, U$6.E
- net LED_B: now also U$5.B
- net LED_G: now also U$6.B
- net LED_R: now also U$3.B
- net N$31: now also R2.1; no longer R28.1
Other:
- moved on the sheet: R1, RESET, SW1, SW2, U1

Commit message: Movingn to PC
Parts:
- added C1, C2: 24pF, MICROCONTROLLER:CAPACITOR
- added C10, C11, C12, C13, C14, C5, C6, C9: .1uF, MICROCONTROLLER:CAPACITOR
- added C3, C4: 10pF, MICROCONTROLLER:CAPACITOR
- added C7: 1uF, MICROCONTROLLER:CAPACITOR
- added C8: 2.2uF, MICROCONTROLLER:CAPACITOR
- added R6: 1M, MICROCONTROLLER:RESISTOR
- added SW3: (no value), MICROCONTROLLER:JS202011SCQN
- added U3: 3.3V, SparkFun-IC-Power:V_REG_AP2112K-3.3V
- added Y2: Y2, MICROCONTROLLER:16MHZ_OSCILLATOR
- U$8: device MICROCONTROLLER:CAPACITOR -> MICROCONTROLLER:USBMICRO
- U$9: device MICROCONTROLLER:CAPACITOR -> MICROCONTROLLER:POWER
- renumbered U$7 to Y1
Connections:
- removed net +MCU_PWR: R2.2
- removed net RST: U$2.RST
- new net !RST: R2.1, RESET.0@A, RESET.0@B, U$2.RST, U1.!RST
- new net +3V3: C10.2, C11.2, C12.2, C13.2, C14.2, C9.2, R2.2, U$2.3V3, U1.VBAT, U1.VDD, U1.VDDA, U1.VDD_2, U1.VDD_3, U1.VDD_4, U3.OUT
- new net N$41: C3.2, U1.XOSC0, Y2.2
- new net N$42: C4.1, U1.XOSC1, Y2.1
- new net N$44: SW3.1, U$8.1
- new net VDDC: C5.2, C6.2, C7.2, C8.2, U1.VDDC, U1.VDDC_2
- net !WAKE: now also R6.2, U1.!WAKE
- net +VBUS: now also R6.1, SW3.2, U$1.VBUS, U$9.+VBUS, U3.EN, U3.IN
- net GND: now also C10.1, C11.1, C12.1, C13.1, C14.1, C3.1, C4.2, C5.1, C6.1, C7.1, C8.1, C9.1, U$1.GND, U$2.GND, U$8.GND@1, U$8.GND@2, U$8.GND@3, U$8.GND@4, U$8.GND@5, U$9.GND, U1.GND, U1.GNDA, U1.GND_2, U1.GND_3, U1.GND_4
- net N$31: now also U3.GND; no longer R2.1, RESET.0@A, RESET.0@B
- net N$38: now also C1.1; no longer U$8.1
- net N$39: now also C2.2; no longer U$9.2
- net N$40: now also C1.2, C2.1; no longer U$8.2, U$9.1
Other:
- moved on the sheet: R2, RESET, U1

Commit message: Started on the Fill Control Design, finished with dev MCU
Parts:
- removed U$8: (no value), MICROCONTROLLER:USBMICRO
- removed U$9: (no value), MICROCONTROLLER:POWER
- added DEBUG: (no value), MICROCONTROLLER:JTAG
- added J1: (no value), MICROCONTROLLER:HEADER_J1
- added J3: (no value), MICROCONTROLLER:USBMICRO
- added PWR: (no value), MICROCONTROLLER:LED_511
- added R7: 10k, MICROCONTROLLER:RESISTOR
- added VBUS: (no value), MICROCONTROLLER:POWER
- R2: value 10k -> 330
- R4, R5: value 330 -> (none)
- U$1: value (none) -> LOGO; device MICROCONTROLLER:HEADER_J1 -> MICROCONTROLLER:LOGO
- renumbered U$2 to J2, U$3 to Q1, U$4 to LED, U$5 to Q2, U$6 to Q3
Connections:
- removed net N$1: U$1.PA2, U1.PA2/SSI0CLK
- removed net N$2: U$1.PA3, U1.PA3/SSI0FSS
- removed net N$27 (its old number): J2.PE2, U1.PE2
- removed net N$28 (its old number): J2.PE3, U1.PE3
- removed net N$44: SW3.1, U$8.1
- new net +VBUS_IN: J3.1, SW3.1, VBUS.+VBUS
- new net N$19: J2.PD5, U1.PD5
- new net N$21: J2.PB0, U1.PB0/USB0ID
- new net N$22: J2.PB1, U1.PB1/USB0VBUS
- new net N$23: J2.PB2, U1.PB2/I2C0SCL
- new net N$43: DEBUG.U0RX, U1.PA0/U0RX
- new net N$45: DEBUG.U0TX, U1.PA1/U0TX
- new net N$46: DEBUG.TCK/SWCLK, U1.PC0/TCK/SWCLK
- new net N$47: DEBUG.TMS/SWDIO, U1.PC1/TMS/SWDIO
- new net N$48: DEBUG.TDI, U1.PC2/TDI
- new net N$49: DEBUG.TDO/SWO, U1.PC3/TDO/SWO
- new net PB6: J1.PB6, U1.PB6
- new net PB7: J1.PB7, U1.PB7
- net !RST: now also R5.1, RESET.1, RESET.2; no longer J2.RST, R2.1, RESET.0@A, RESET.0@B
- net !WAKE: now also R4.1; no longer R1.1
- net +3V3: now also J1.3V3, R5.2; no longer J2.3V3, R2.2
- net +VBUS: now also J1.VBUS, PWR.2; no longer U$1.VBUS, U$9.+VBUS
- net GND: now also J1.GND, J3.GND@1, J3.GND@2, J3.GND@3, J3.GND@4, J3.GND@5, R7.1, RESET.3, RESET.4, SW1.3, SW1.4, SW2.3, SW2.4, U3.GND, VBUS.GND; no longer J2.GND, RESET.1@A, RESET.1@B, SW1.1@A, SW1.1@B, SW2.1@A, SW2.1@B, U$1.GND, U$8.GND@1, U$8.GND@2, U$8.GND@3, U$8.GND@4, U$8.GND@5, U$9.GND
- net N$10: now also J1.PC5, U1.PC5; no longer U$1.PB3, U1.PB3/I2C0SDA
- net N$11: now also J1.PC4, U1.PC4; no longer U$1.PB4, U1.PB4
- net N$12: now also J1.PA2, U1.PA2/SSI0CLK; no longer U$1.PB5, U1.PB5
- net N$13: now also J1.PA3, U1.PA3/SSI0FSS; no longer U$1.PB6, U1.PB6
- net N$14: now also J1.PA4, U1.PA4/SSI0RX; no longer U$1.PB7, U1.PB7
- net N$15: now also J1.PA5, U1.PA5/SSI0TX; no longer U$1.PC4, U1.PC4
- net N$16: now also J1.PA6, U1.PA6; no longer U$1.PC5, U1.PC5
- net N$17: now also J1.PA7, U1.PA7; no longer U$1.PC6, U1.PC6
- net N$18: now also J2.PD4, U1.PD4; no longer U$1.PC7, U1.PC7
- net N$24: now also J2.PB3, U1.PB3/I2C0SDA; no longer J2.PD7, U1.PD7
- net N$25: now also J2.PB4, U1.PB4; no longer J2.PE0, U1.PE0
- net N$26: now also J2.PB5, U1.PB5; no longer J2.PE1, U1.PE1
- net N$3: now also J1.PE3, U1.PE3; no longer U$1.PA4, U1.PA4/SSI0RX
- net N$31: now also PWR.1, R7.2; no longer U3.GND
- net N$32: now also R1.2; no longer R3.2
- net N$33: now also R2.2; no longer R4.2
- net N$34: now also R3.2; no longer R5.2
- net N$35: now also R3.1; no longer R5.1
- net N$36: now also R2.1; no longer R4.1
- net N$37: now also R1.1; no longer R3.1
- net N$4: now also J1.PE2, U1.PE2; no longer U$1.PA5, U1.PA5/SSI0TX
- net N$5: now also J1.PE1, U1.PE1; no longer U$1.PA6, U1.PA6
- net N$6: now also J1.PE0, U1.PE0; no longer U$1.PA7, U1.PA7
- net N$7: now also J1.PD7, U1.PD7; no longer U$1.PB0, U1.PB0/USB0ID
- net N$8: now also J1.PC7, U1.PC7; no longer U$1.PB1, U1.PB1/USB0VBUS
- net N$9: now also J1.PC6, U1.PC6; no longer U$1.PB2, U1.PB2/I2C0SCL
- net SW1: now also SW1.1, SW1.2; no longer SW1.0@A, SW1.0@B
- net SW2: now also R4.2, SW2.1, SW2.2; no longer R1.2, SW2.0@A, SW2.0@B
Other:
- moved on the sheet: R1, R2, R3, R4, R5, SW3, U3

Commit message: starting on final
Parts:
- removed U$1: LOGO, MICROCONTROLLER:LOGO
Changed lines of the file:
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@@
 <part name="GND13" library="audio amplifier example" library_urn="urn:adsk.eagle:library:970892" deviceset="GND" device="" value="SUP"/>
 <part name="J3" library="MICROCONTROLLER" deviceset="USBMICRO" device=""/>
-<part name="U$1" library="MICROCONTROLLER" deviceset="LOGO" device=""/>
 </parts>
 <sheets>
