File: EE474FINAL/EE474FINAL/EE474FINAL.sch (EAGLE design)
At the start: 24 parts, among them U1 TM4C123_DEVICE, U4 3.3V

Commit message: Ready for layout
Parts:
- removed S2: (no value), MICROCONTROLLER:DRV8825
- removed U$1: (no value), FillControl:OPTOISOLATOR
- added C10: 2.2uF, MICROCONTROLLER:CAPACITOR
- added C11, C12, C13, C14, C15, C16, C7, C8: .1uF, MICROCONTROLLER:CAPACITOR
- added C3, C4: 24pF, MICROCONTROLLER:CAPACITOR
- added C5, C6: 10pF, MICROCONTROLLER:CAPACITOR
- added C9: 1uF, MICROCONTROLLER:CAPACITOR
- added GND, PA2, PA3, PA4, PA5: (no value), MICROCONTROLLER:TESTPOINT
- added J5, J6: (no value), MICROCONTROLLER:4POS_MOLEXVERT
- added J7: (no value), MICROCONTROLLER:6POS_JST
- added R5, R7, R8: (no value), rcl:R-US_R0402
- added R6: 1M, MICROCONTROLLER:RESISTOR
- added SA, SB: (no value), MICROCONTROLLER:DRV8825
- added U7: (no value), FillControl:OPTOISOLATOR
- added Y1: 32kHz, MICROCONTROLLER:32KHZ_OSCILATOR
- added Y2: Y2, MICROCONTROLLER:16MHZ_OSCILLATOR
- S1: device MICROCONTROLLER:DRV8825 -> MICROCONTROLLER:SLIDESWITCH
Connections:
- removed net +24V: F1.1, J1.+24V
- removed net +VBUS: U4.EN, U4.IN
- new net !RST: U1.!RST
- new net !WAKE: R6.2, U1.!WAKE
- new net +20V: F1.1, S1.2, SA.VMOT, SB.VMOT
- new net BAT: R5.2, R7.1, U1.PE3
- new net CTS: U2.UART_CTS
- new net DIR_A: SA.DIR, U1.PD4
- new net DIR_B: SB.DIR, U1.PF4
- new net M0_A: SA.M0, U1.PD0
- new net M0_B: SB.M0, U1.PF0
- new net M1_A: SA.M1, U1.PD1
- new net M1_B: SB.M1, U1.PF1
- new net M2_A: SA.M2, U1.PD2
- new net M2_B: SB.M2, U1.PF2
- new net N$10: J5.GRN, SA.B1
- new net N$11: J5.BLK, SA.B2
- new net N$12: J6.BLU, SB.A2
- new net N$13: J6.RED, SB.A1
- new net N$14: J6.GRN, SB.B1
- new net N$15: J6.BLK, SB.B2
- new net N$16: SB.!RST, SB.!SLP
- new net N$17: SA.!RST, SA.!SLP
- new net N$19: J1.+20V, S1.1
- new net N$20: R8.1, U6.C
- new net N$21: PA3.P$1, U1.PA3/SSI0FSS
- new net N$38: C3.1, U1.OSC0, Y1.2
- new net N$39: C4.2, U1.OSC1, Y1.1
- new net N$40: C3.2, C4.1, U1.GNDX
- new net N$41: C5.2, U1.XOSC0, Y2.2
- new net N$42: C6.1, U1.XOSC1, Y2.1
- new net N$8: J5.BLU, SA.A2
- new net N$9: J5.RED, SA.A1
- new net PA2: PA2.P$1, U1.PA2/SSI0CLK
- new net PA4: PA4.P$1, U1.PA4/SSI0RX
- new net PA5: PA5.P$1, U1.PA5/SSI0TX
- new net RTS: U2.UART_RTS
- new net RX-1: U1.PB1/USB0VBUS, U2.UART_RX
- new net RXD: J7.1, U1.PA0/U0RX
- new net STEP_A: SA.STEP, U1.PD3
- new net STEP_B: SB.STEP, U1.PF3
- new net TCK: J7.3, U1.PC0/TCK/SWCLK
- new net TDI: J7.5, U1.PC2/TDI
- new net TDO: J7.6, U1.PC3/TDO/SWO
- new net TMS: J7.4, U1.PC1/TMS/SWDIO
- new net TX-0: U1.PB0/USB0ID, U2.UART_TX
- new net TXD: J7.2, U1.PA1/U0TX
- new net VDDC: C10.2, C7.2, C8.2, C9.2, U1.VDDC, U1.VDDC_2
- net +3V3: now also C11.2, C12.2, C13.2, C14.2, C15.2, C16.2, SA.!FLT, SB.!FLT, U1.VBAT, U1.VDD, U1.VDDA, U1.VDD_2, U1.VDD_3, U1.VDD_4, U2.VDD
- net +5V: now also R6.1, U4.EN, U4.IN
- net BUZZER: now also U1.PA6
- net FAN: now also U1.PA7
- net GND: now also C10.1, C11.1, C12.1, C13.1, C14.1, C15.1, C16.1, C5.1, C6.2, C7.1, C8.1, C9.1, GND.P$1, R5.1, S1.GND, SA.GND, SB.GND, U1.GND, U1.GNDA, U1.GND_2, U1.GND_3, U1.GND_4, U2.GND
- net LT: now also U1.PE2
- net N$3: now also U7.4; no longer U$1.4
- net N$4: now also U7.3; no longer U$1.3
- net N$5: now also R8.2; no longer U6.C
- net N$6: now also U7.2; no longer U$1.2
- net TRIG: now also U1.PB5, U7.1; no longer U$1.1
- net VIN: now also R7.2
Other:
- moved on the sheet: C1, C2, D1, F1, J2, J3, J4, L1, R1, R2, R3, R4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

Commit message: to pc
Parts:
- added GREEN, RED: (no value), MICROCONTROLLER:LED_511
- added R10, R11, R12, R9: (no value), MICROCONTROLLER:RESISTOR
- added RESET: (no value), MICROCONTROLLER:SWITCH_B3S
Connections:
- net N$38 renamed OSC0
- net N$39 renamed OSC1
- net N$40 renamed GNDX
- net N$41 renamed XOSC0
- net N$42 renamed XOSC1
- new net N$18: RED.2, U2.GPIO5
- new net N$22: R10.2, RED.1
- new net N$23: GREEN.1, R11.2
- new net N$24: GREEN.2, U2.GPIO2
- new net N$25: R12.2, U2.GPIO4
- net !RST: now also R9.1, RESET.1, RESET.2
- net +3V3: now also R9.2
- net GND: now also R10.1, R11.1, R12.1, RESET.3, RESET.4
Other:
- moved on the sheet: U2

Commit message: to surface
Parts:
- added C17: (no value), FillControl:CAP_18
- D1: value (none) -> DIODE_SHOTKY_SMA; device FillControl:SHOTKEY -> MICROCONTROLLER:DIODE_SHOTKY_SMA
- J1: device MICROCONTROLLER:2POS_MOLEX -> MICROCONTROLLER:2POS_JSTVERT_2.5
- J3, J4: device MICROCONTROLLER:2POS_JST -> MICROCONTROLLER:2POS_JSTVERT_2.0
- J6: device MICROCONTROLLER:4POS_MOLEXVERT -> MICROCONTROLLER:4POS_MOLEX_2.54
Connections:
- net N$19 renamed 20IN
- net N$5 renamed FAN_OUT
- removed net N$15: J6.BLK, SB.B2
- new net N$5: J6.BLK, SB.A2
- net +20V: now also C17.1
- net BUZZER: now also U1.PB7; no longer U1.PA6
- net DIR_A: now also U1.PA2/SSI0CLK; no longer U1.PD4
- net FAN: now also U1.PB6; no longer U1.PA7
- net GND: now also C17.2, S1.3
- net M0_A: now also U1.PA6; no longer U1.PD0
- net M1_A: now also U1.PA5/SSI0TX; no longer U1.PD1
- net M2_A: now also U1.PA4/SSI0RX; no longer U1.PD2
- net N$12: now also J6.GRN, SB.A1; no longer J6.BLU, SB.A2
- net N$13: now also SB.B1; no longer SB.A1
- net N$14: now also J6.BLU, SB.B2; no longer J6.GRN, SB.B1
- net N$21: now also U1.PC6; no longer U1.PA3/SSI0FSS
- net PA2: now also U1.PC7; no longer U1.PA2/SSI0CLK
- net PA4: now also U1.PC5; no longer U1.PA4/SSI0RX
- net PA5: now also U1.PC4; no longer U1.PA5/SSI0TX
- net STEP_A: now also U1.PA3/SSI0FSS; no longer U1.PD3
Other:
- moved on the sheet: GND, PA2, PA3, PA4, PA5

Commit message: merge
Parts:
- removed PA2, PA3, PA4, PA5: (no value), MICROCONTROLLER:TESTPOINT
- added PD0, PD1, PD2, PE5: (no value), MICROCONTROLLER:TESTPOINT
- renumbered GREEN to CON, RED to DIS
Connections:
- removed net N$21: PA3.P$1, U1.PC6
- removed net PA2: PA2.P$1, U1.PC7
- removed net PA4: PA4.P$1, U1.PC5
- removed net PA5: PA5.P$1, U1.PC4
- new net PD0: PD0.P$1, U1.PD0
- new net PD1: PD1.P$1, U1.PD1
- new net PD2: PD2.P$1, U1.PD2
- new net PE5: PE5.P$1, U1.PE5
- net BUZZER: now also U1.PC4; no longer U1.PB7
- net DIR_B: now also U1.PA7; no longer U1.PF4
- net FAN: now also U1.PC5; no longer U1.PB6
- net M0_B: now also U1.PF3; no longer U1.PF0
- net M1_B: now also U1.PF2; no longer U1.PF1
- net M2_B: now also U1.PF1; no longer U1.PF2
- net STEP_B: now also U1.PF0; no longer U1.PF3
- net TRIG: now also U1.PD3; no longer U1.PB5

Commit message: done
Parts:
- added ENDSTOP: (no value), MICROCONTROLLER:2POS_JSTVERT_2.0
- added R13: (no value), MICROCONTROLLER:RESISTOR
- renumbered J3 to LIGHT, J4 to FAN, J7 to DEBUG, SG1 to SPKR
Connections:
- new net N$15: ENDSTOP.1, R13.1, U1.PE4
- net +3V3: now also R13.2
- net GND: now also ENDSTOP.2
Changed lines of the file:
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@@
 <part name="SA" library="MICROCONTROLLER" deviceset="DRV8825" device=""/>
 <part name="SB" library="MICROCONTROLLER" deviceset="DRV8825" device=""/>
-<part name="SG1" library="buzzer" library_urn="urn:adsk.eagle:library:113" deviceset="F/QMBIII" device="" package3d_urn="urn:adsk.eagle:package:5267/1"/>
+<part name="SPKR" library="buzzer" library_urn="urn:adsk.eagle:library:113" deviceset="F/QMBIII" device="" package3d_urn="urn:adsk.eagle:package:5267/1"/>
 <part name="GND11" library="audio amplifier example" library_urn="urn:adsk.eagle:library:970892" deviceset="GND" device="" value="SUP"/>
 <part name="U4" library="SparkFun-IC-Power" library_urn="urn:adsk.eagle:library:526" deviceset="V_REG_AP2112" device="K-3.3V" package3d_urn="urn:adsk.eagle:package:39060/1" value="3.3V"/>
@@
 <part name="GND9" library="audio amplifier example" library_urn="urn:adsk.eagle:library:970892" deviceset="GND" device="" value="SUP"/>
 <part name="GND10" library="audio amplifier example" library_urn="urn:adsk.eagle:library:970892" deviceset="GND" device="" value="SUP"/>
-<part name="J7" library="MICROCONTROLLER" deviceset="6POS_JST" device=""/>
+<part name="DEBUG" library="MICROCONTROLLER" deviceset="6POS_JST" device=""/>
 <part name="S1" library="MICROCONTROLLER" deviceset="SLIDESWITCH" device=""/>
 <part name="R5" library="rcl" library_urn="urn:adsk.eagle:library:334" deviceset="R-US_" device="R0402" package3d_urn="urn:adsk.eagle:package:23547/3"/>
@@
 <part name="R12" library="MICROCONTROLLER" deviceset="RESISTOR" device="" package3d_urn="urn:adsk.eagle:package:14416342/1"/>
 <part name="SUPPLY5" library="supply2" library_urn="urn:adsk.eagle:library:372" deviceset="GND" device=""/>
-<part name="J3" library="MICROCONTROLLER" deviceset="2POS_JSTVERT_2.0" device=""/>
-<part name="J4" library="MICROCONTROLLER" deviceset="2POS_JSTVERT_2.0" device=""/>
+<part name="LIGHT" library="MICROCONTROLLER" deviceset="2POS_JSTVERT_2.0" device=""/>
+<part name="FAN" library="MICROCONTROLLER" deviceset="2POS_JSTVERT_2.0" device=""/>
 <part name="J1" library="MICROCONTROLLER" deviceset="2POS_JSTVERT_2.5" device=""/>
 <part name="D1" library="MICROCONTROLLER" deviceset="DIODE_SHOTKY_SMA" device=""/>
@@
 <part name="PD0" library="MICROCONTROLLER" deviceset="TESTPOINT" device=""/>
 <part name="PE5" library="MICROCONTROLLER" deviceset="TESTPOINT" device=""/>
+<part name="R13" library="MICROCONTROLLER" deviceset="RESISTOR" device="" package3d_urn="urn:adsk.eagle:package:14416342/1"/>
+<part name="ENDSTOP" library="MICROCONTROLLER" deviceset="2POS_JSTVERT_2.0" device=""/>
+<part name="GND14" library="audio amplifier example" library_urn="urn:adsk.eagle:library:970892" deviceset="GND" device="" value="SUP"/>
 </parts>
 <sheets>
@@
 <instance part="GND9" gate="G$1" x="251.46" y="104.14" smashed="yes"/>
 <instance part="GND10" gate="G$1" x="205.74" y="71.12" smashed="yes"/>
-<instance part="J7" gate="A" x="134.62" y="182.88" smashed="yes" rot="MR0">
+<instance part="DEBUG" gate="A" x="134.62" y="182.88" smashed="yes" rot="MR0">
 <attribute name="NAME" x="134.62" y="189.23" size="2.54" layer="95" rot="MR0"/>
 </instance>
@@
 <attribute name="NAME" x="237.998" y="179.324" size="1.778" layer="94" rot="MR0"/>
 </instance>
+<instance part="R13" gate="&gt;NAME" x="243.84" y="177.8" smashed="yes" rot="MR90">
+<attribute name="NAME" x="246.1006" y="176.022" size="1.778" layer="95" rot="MR90"/>
+<attribute name="VALUE" x="240.538" y="175.514" size="1.778" layer="96" rot="MR90"/>
+</instance>
+<instance part="ENDSTOP" gate="A" x="248.92" y="167.64" smashed="yes">
+<attribute name="NAME" x="251.46" y="175.26" size="1.778" layer="95"/>
+</instance>
+<instance part="GND14" gate="G$1" x="243.84" y="165.1" smashed="yes"/>
 </instances>
 <busses>
@@
 <pinref part="R12" gate="&gt;NAME" pin="1"/>
 <wire x1="96.52" y1="137.16" x2="96.52" y2="139.7" width="0.1524" layer="91"/>
+</segment>
+<segment>
+<pinref part="ENDSTOP" gate="A" pin="2"/>
+<wire x1="248.92" y1="167.64" x2="243.84" y2="167.64" width="0.1524" layer="91"/>
+<wire x1="243.84" y1="167.64" x2="243.84" y2="165.1" width="0.1524" layer="91"/>
+<pinref part="GND14" gate="G$1" pin="GND"/>
 </segment>
 </net>
@@
 <label x="104.14" y="67.564" size="1.778" layer="95" rot="MR0"/>
 </segment>
+<segment>
+<pinref part="R13" gate="&gt;NAME" pin="2"/>
+<wire x1="243.84" y1="182.88" x2="243.84" y2="185.42" width="0.1524" layer="91"/>
+<label x="243.84" y="185.42" size="1.778" layer="95"/>
+</segment>
 </net>
 <net name="TX-0" class="0">
@@
 <net name="RXD" class="0">
 <segment>
-<pinref part="J7" gate="A" pin="1"/>
+<pinref part="DEBUG" gate="A" pin="1"/>
 <pinref part="U1" gate="A" pin="PA0/U0RX"/>
 <wire x1="139.7" y1="185.42" x2="154.94" y2="185.42" width="0.1524" layer="91"/>
@@
 <segment>
 <pinref part="U1" gate="A" pin="PA1/U0TX"/>
-<pinref part="J7" gate="A" pin="2"/>
+<pinref part="DEBUG" gate="A" pin="2"/>
 <wire x1="154.94" y1="182.88" x2="139.7" y2="182.88" width="0.1524" layer="91"/>
 <label x="144.78" y="182.88" size="1.778" layer="95"/>
@@
 <net name="TCK" class="0">
 <segment>
-<pinref part="J7" gate="A" pin="3"/>
+<pinref part="DEBUG" gate="A" pin="3"/>
 <pinref part="U1" gate="A" pin="PC0/TCK/SWCLK"/>
 <wire x1="139.7" y1="180.34" x2="154.94" y2="180.34" width="0.1524" layer="91"/>
@@
 <segment>
 <pinref part="U1" gate="A" pin="PC1/TMS/SWDIO"/>
-<pinref part="J7" gate="A" pin="4"/>
+<pinref part="DEBUG" gate="A" pin="4"/>
 <wire x1="154.94" y1="177.8" x2="139.7" y2="177.8" width="0.1524" layer="91"/>
 <label x="144.78" y="177.8" size="1.778" layer="95"/>
@@
 <net name="TDI" class="0">
 <segment>
-<pinref part="J7" gate="A" pin="5"/>
+<pinref part="DEBUG" gate="A" pin="5"/>
 <pinref part="U1" gate="A" pin="PC2/TDI"/>
 <wire x1="139.7" y1="175.26" x2="154.94" y2="175.26" width="0.1524" layer="91"/>
@@
 <segment>
 <pinref part="U1" gate="A" pin="PC3/TDO/SWO"/>
-<pinref part="J7" gate="A" pin="6"/>
+<pinref part="DEBUG" gate="A" pin="6"/>
 <wire x1="154.94" y1="172.72" x2="139.7" y2="172.72" width="0.1524" layer="91"/>
 <label x="144.78" y="172.72" size="1.778" layer="95"/>
@@
 <label x="210.82" y="182.88" size="1.778" layer="95"/>
 <pinref part="U1" gate="A" pin="PD3"/>
+</segment>
+</net>
+<net name="N$15" class="0">
+<segment>
+<pinref part="U1" gate="A" pin="PE4"/>
+<wire x1="205.74" y1="170.18" x2="243.84" y2="170.18" width="0.1524" layer="91"/>
+<wire x1="243.84" y1="170.18" x2="243.84" y2="172.72" width="0.1524" layer="91"/>
+<pinref part="R13" gate="&gt;NAME" pin="1"/>
+<pinref part="ENDSTOP" gate="A" pin="1"/>
+<wire x1="243.84" y1="170.18" x2="248.92" y2="170.18" width="0.1524" layer="91"/>
+<junction x="243.84" y="170.18"/>
 </segment>
 </net>
@@
 <attribute name="NAME" x="55.626" y="80.01" size="2.54" layer="95"/>
 </instance>
-<instance part="SG1" gate="G$1" x="254" y="165.1" smashed="yes" rot="MR90">
+<instance part="SPKR" gate="G$1" x="254" y="165.1" smashed="yes" rot="MR90">
 <attribute name="NAME" x="260.35" y="162.56" size="1.778" layer="95" rot="MR90"/>
 </instance>
@@
 <attribute name="VALUE" x="254.762" y="90.17" size="1.778" layer="96" rot="R90"/>
 </instance>
-<instance part="J3" gate="A" x="180.34" y="114.3" smashed="yes">
+<instance part="LIGHT" gate="A" x="180.34" y="114.3" smashed="yes">
 <attribute name="NAME" x="182.88" y="121.92" size="1.778" layer="95"/>
 </instance>
-<instance part="J4" gate="A" x="251.46" y="104.14" smashed="yes">
+<instance part="FAN" gate="A" x="251.46" y="104.14" smashed="yes">
 <attribute name="NAME" x="254" y="111.76" size="1.778" layer="95"/>
 </instance>
@@
 <net name="+5V" class="0">
 <segment>
-<pinref part="SG1" gate="G$1" pin="-"/>
+<pinref part="SPKR" gate="G$1" pin="-"/>
 <wire x1="251.46" y1="170.18" x2="251.46" y2="177.8" width="0.1524" layer="91"/>
 <label x="248.92" y="177.8" size="1.778" layer="95"/>
@@
 <wire x1="251.46" y1="106.68" x2="251.46" y2="114.3" width="0.1524" layer="91"/>
 <label x="248.92" y="114.3" size="1.778" layer="95"/>
-<pinref part="J4" gate="A" pin="1"/>
+<pinref part="FAN" gate="A" pin="1"/>
 </segment>
 <segment>
@@
 <wire x1="180.34" y1="116.84" x2="180.34" y2="129.54" width="0.1524" layer="91"/>
 <label x="177.8" y="129.54" size="1.778" layer="95"/>
-<pinref part="J3" gate="A" pin="1"/>
+<pinref part="LIGHT" gate="A" pin="1"/>
 </segment>
 <segment>
@@
 <net name="N$2" class="0">
 <segment>
-<pinref part="SG1" gate="G$1" pin="+"/>
+<pinref part="SPKR" gate="G$1" pin="+"/>
 <pinref part="U5" gate="G$1" pin="C"/>
 <wire x1="251.46" y1="162.56" x2="251.46" y2="154.94" width="0.1524" layer="91"/>
@@
 <wire x1="180.34" y1="114.3" x2="172.72" y2="114.3" width="0.1524" layer="91"/>
 <label x="170.18" y="114.3" size="1.778" layer="95"/>
-<pinref part="J3" gate="A" pin="2"/>
+<pinref part="LIGHT" gate="A" pin="2"/>
 <junction x="180.34" y="114.3"/>
 </segment>
@@
 <pinref part="R8" gate="G$1" pin="2"/>
 <wire x1="251.46" y1="99.06" x2="251.46" y2="104.14" width="0.1524" layer="91"/>
-<pinref part="J4" gate="A" pin="2"/>
-</segment>
-</net>
+<pinref part="FAN" gate="A" pin="2"/>
+</segment>
+</net>

Commit message: fixing...
Connections:
- net GND: now also U3.6
Changed lines of the file:
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@@
 <wire x1="157.48" y1="160.02" x2="157.48" y2="154.94" width="0.1524" layer="91"/>
 <wire x1="137.16" y1="157.48" x2="137.16" y2="154.94" width="0.1524" layer="91"/>
-<wire x1="137.16" y1="154.94" x2="157.48" y2="154.94" width="0.1524" layer="91"/>
+<wire x1="137.16" y1="154.94" x2="142.24" y2="154.94" width="0.1524" layer="91"/>
 <pinref part="U3" gate="A" pin="GND"/>
+<wire x1="142.24" y1="154.94" x2="157.48" y2="154.94" width="0.1524" layer="91"/>
 <wire x1="96.52" y1="172.72" x2="96.52" y2="154.94" width="0.1524" layer="91"/>
 <wire x1="96.52" y1="154.94" x2="119.38" y2="154.94" width="0.1524" layer="91"/>
@@
 <wire x1="73.66" y1="160.02" x2="73.66" y2="154.94" width="0.1524" layer="91"/>
 <junction x="73.66" y="154.94"/>
+<pinref part="U3" gate="A" pin="6"/>
+<wire x1="134.62" y1="175.26" x2="142.24" y2="175.26" width="0.1524" layer="91"/>
+<wire x1="142.24" y1="175.26" x2="142.24" y2="154.94" width="0.1524" layer="91"/>
+<junction x="142.24" y="154.94"/>
 </segment>
 <segment>
