File: EE474FINAL/EE474FINAL/EE474FINAL.brd (EAGLE design)
At the start: 160 x 100 mm, 53 parts, among them U1 TM4C123_DEVICE, U4 3.3V, Y1 32kHz, Y2 Y2

Commit message: to pc
Parts:
- added GREEN, RED: (no value), MICROCONTROLLER:LED_511
- added R10, R11, R12, R9: (no value), MICROCONTROLLER:CAPC1005X35N
- added RESET: (no value), MICROCONTROLLER:SW_BS3
- moved C16 143.7 mm to (64.1, 61.4), flipped to the bottom, turned to 90 degrees
- moved C15 140.1 mm to (65.4, 60.2), flipped to the bottom, turned to 180 degrees
- moved C14 135.5 mm to (65.4, 57.0), flipped to the bottom, turned to 180 degrees
- moved C13 129.6 mm to (64.2, 55.4), flipped to the bottom, turned to 270 degrees
- moved C12 118.7 mm to (58.8, 58.8), flipped to the bottom
- moved C6 118.1 mm to (77.7, 54.4), turned to 180 degrees
- moved C11 113.5 mm to (58.8, 59.8), flipped to the bottom
- moved C8 110.2 mm to (59.7, 55.3), flipped to the bottom, turned to 270 degrees
- moved C5 109.4 mm to (73.9, 54.4), turned to 180 degrees
- moved C7 106.2 mm to (60.7, 55.3), flipped to the bottom, turned to 270 degrees
- moved C4 102.9 mm to (73.5, 60.4), turned to 90 degrees
- moved C3 98.2 mm to (73.5, 58.4), turned to 90 degrees
- moved C10 78.9 mm to (60.7, 61.4), flipped to the bottom, turned to 90 degrees
- moved C9 78.2 mm to (59.7, 61.4), flipped to the bottom, turned to 90 degrees
- moved Y2 19.5 mm to (75.8, 50.7), turned to 180 degrees
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Connections:
- net N$38 renamed OSC0
- net N$39 renamed OSC1
- net N$40 renamed GNDX
- net N$41 renamed XOSC0
- net N$42 renamed XOSC1
- new net N$18: RED.P$2, U2.21
- new net N$22: R10.2, RED.P$1
- new net N$23: GREEN.P$1, R11.2
- new net N$24: GREEN.P$2, U2.19
- new net N$25: R12.2, U2.22
- net !RST: now also R9.1, RESET.1, RESET.2
- net +3V3: now also R9.2
- net GND: now also R10.1, R11.1, R12.1, RESET.3, RESET.4
Routing:
- net +3V3: track 0.00 -> 37.3 mm, vias 0 -> 6
- net GND: track 0.00 -> 23.2 mm, vias 0 -> 5
- net !RST: track 0.00 -> 20.2 mm
- net XOSC1: track 0.00 -> 15.1 mm
- net VDDC: track 0.00 -> 9.73 mm, vias 0 -> 2
- net GNDX: track 0.00 -> 9.37 mm, vias 0 -> 2
- net XOSC0: track 0.00 -> 9.13 mm
- net OSC1: track 0.00 -> 8.23 mm
- net OSC0: track 0.00 -> 7.51 mm
- net DIR_A: track 0.00 -> 4.96 mm
- net TX-0: track 0.00 -> 4.63 mm
- net RX-1: track 0.00 -> 4.23 mm

Commit message: to surface
Parts:
- added C17: (no value), FillControl:CAP_ULH_10X10
- D1: value (none) -> DIODE_SHOTKY_SMA; device FillControl:SMC -> MICROCONTROLLER:SMA
- J1: device MICROCONTROLLER:2POS_MOLEX -> MICROCONTROLLER:2POS_JSTVERT
- J3, J4: device MICROCONTROLLER:JST_S2B-PH-K-S(LF)(SN) -> MICROCONTROLLER:2POS_JSTVERT_2.00
- J6: device MICROCONTROLLER:4POS_MOLEXVERT -> MICROCONTROLLER:MOLEX_0705530003
- moved R7 135.9 mm to (73.6, 63.7)
- moved PA5 134.7 mm to (55.8, 62.5)
- moved PA4 134.4 mm to (58.0, 62.5)
- moved PA3 134.1 mm to (60.2, 62.5)
- moved PA2 133.9 mm to (62.5, 62.5)
- moved R5 129.0 mm to (70.4, 63.7)
- moved R2 126.6 mm to (79.2, 61.8), turned to 90 degrees
- moved R8 113.6 mm to (48.7, 87.5), turned to 90 degrees
- moved R4 112.6 mm to (58.7, 71.4), turned to 90 degrees
- moved GND 109.8 mm to (40.5, 61.9), flipped to the bottom, turned to 90 degrees
- moved R1 98.0 mm to (54.5, 65.0)
- moved R3 96.4 mm to (46.7, 77.5), turned to 90 degrees
- moved TP1 92.9 mm to (8.20, 53.5), turned to 90 degrees
- moved R6 73.6 mm to (51.2, 61.8)
- moved J4 73.5 mm to (43.5, 90.2)
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Connections:
- net N$19 renamed 20IN
- net N$5 renamed FAN_OUT
- removed net N$15: J6.P$1, SB.B2
- new net N$5: J6.4, SB.A2
- net +20V: now also C17.1
- net BUZZER: now also U1.4; no longer U1.23
- net DIR_A: now also U1.19; no longer U1.43
- net FAN: now also U1.1; no longer U1.24
- net GND: now also C17.2, S1.3
- net M0_A: now also U1.23; no longer U1.61
- net M1_A: now also U1.22; no longer U1.62
- net M2_A: now also U1.21; no longer U1.63
- net N$12: now also J6.3, SB.A1; no longer J6.P$4, SB.A2
- net N$13: now also J6.2, SB.B1; no longer J6.P$3, SB.A1
- net N$14: now also J6.1, SB.B2; no longer J6.P$2, SB.B1
- net N$21: now also U1.14; no longer U1.20
- net PA2: now also U1.13; no longer U1.19
- net PA4: now also U1.15; no longer U1.21
- net PA5: now also U1.16; no longer U1.22
- net RXD: now also J7.6; no longer J7.1
- net STEP_A: now also U1.20; no longer U1.64
- net TCK: now also J7.4; no longer J7.3
- net TDI: now also J7.2; no longer J7.5
- net TDO: now also J7.1; no longer J7.6
- net TMS: now also J7.3; no longer J7.4
- net TXD: now also J7.5; no longer J7.2
Routing:
- net +20V: track 0.00 -> 174.0 mm, vias 0 -> 1
- net +3V3: track 37.3 -> 154.9 mm, vias 6 -> 7
- net +5V: track 0.00 -> 90.1 mm
- net TXD: track 0.00 -> 43.2 mm, vias 0 -> 2
- net RXD: track 0.00 -> 42.7 mm, vias 0 -> 2
- net LT: track 0.00 -> 39.6 mm, vias 0 -> 1
- net VIN: track 0.00 -> 36.6 mm
- net N$5: track 0.00 -> 29.0 mm
- net N$8: track 0.00 -> 27.7 mm
- net N$12: track 0.00 -> 25.3 mm
- net TCK: track 0.00 -> 25.0 mm
- net TMS: track 0.00 -> 24.6 mm
- net TDI: track 0.00 -> 24.2 mm
- net N$9: track 0.00 -> 24.1 mm
- net TDO: track 0.00 -> 23.8 mm
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Other:
- board size 160 x 100 mm -> 104.8 x 84.8 mm

Commit message: merge
Parts:
- removed GREEN, RED: (no value), MICROCONTROLLER:LED_511
- removed PA2, PA3, PA4, PA5: (no value), MICROCONTROLLER:TESTPOINT
- added CON, DIS: (no value), MICROCONTROLLER:LED_511
- added PD0, PD1, PD2, PE5: (no value), MICROCONTROLLER:TESTPOINT
- moved R11 38.0 mm to (58.9, 28.4)
- moved U3 36.9 mm to (36.0, 59.5)
- moved C10 36.9 mm to (37.8, 42.7)
- moved C11 36.9 mm to (36.1, 44.6)
- moved C12 36.9 mm to (35.1, 44.6)
- moved C8 36.9 mm to (31.6, 43.7)
- moved C9 36.9 mm to (37.8, 43.7)
- moved J1 36.9 mm to (43.9, 75.7)
- moved R4 36.9 mm to (23.7, 59.6)
- moved R9 36.9 mm to (33.8, 26.2)
- moved RESET 36.9 mm to (43.9, 25.9)
- moved SG1 36.9 mm to (11.6, 56.4)
- moved U1 36.9 mm to (34.6, 41.1)
- moved U2 36.9 mm to (52.2, 28.7)
- moved U6 36.9 mm to (20.3, 61.1)
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Connections:
- removed net N$21: PA3.P$1, U1.14
- removed net PA2: PA2.P$1, U1.13
- removed net PA4: PA4.P$1, U1.15
- removed net PA5: PA5.P$1, U1.16
- new net PD0: PD0.P$1, U1.61
- new net PD1: PD1.P$1, U1.62
- new net PD2: PD2.P$1, U1.63
- new net PE5: PE5.P$1, U1.60
- net BUZZER: now also U1.16; no longer U1.4
- net DIR_B: now also U1.24; no longer U1.5
- net FAN: now also U1.15; no longer U1.1
- net M0_B: now also U1.31; no longer U1.28
- net M1_B: now also U1.30; no longer U1.29
- net M2_B: now also U1.29; no longer U1.30
- net N$18: now also DIS.P$2; no longer RED.P$2
- net N$22: now also DIS.P$1; no longer RED.P$1
- net N$23: now also CON.P$1; no longer GREEN.P$1
- net N$24: now also CON.P$2; no longer GREEN.P$2
- net STEP_B: now also U1.28; no longer U1.31
- net TRIG: now also U1.64; no longer U1.57
Routing:
- net +3V3: track 154.9 -> 238.0 mm, vias 7 -> 10
- net M0_B: track 0.00 -> 36.1 mm
- net M1_B: track 0.00 -> 35.6 mm
- net M2_B: track 0.00 -> 35.2 mm
- net DIR_B: track 0.00 -> 30.0 mm
- net STEP_B: track 0.00 -> 29.6 mm
- net FAN: track 0.01 -> 18.4 mm
- net PE5: track 0.00 -> 17.7 mm
- net N$24: track 0.00 -> 14.7 mm, vias 0 -> 1
- net PD0: track 0.00 -> 14.6 mm
- net BUZZER: track 0.00 -> 12.0 mm
- net PD1: track 0.00 -> 11.5 mm
- net !RST: track 17.1 -> 25.6 mm
- net N$18: track 0.00 -> 8.52 mm, vias 0 -> 1
- net PD2: track 0.00 -> 8.23 mm
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Other:
- board size 104.8 x 84.8 mm -> 69.5 x 84.8 mm

Commit message: done
Parts:
- removed J3, J4: (no value), MICROCONTROLLER:2POS_JSTVERT_2.00
- removed J7: (no value), MICROCONTROLLER:6POS_JST
- removed SG1: F/QMBIII, buzzer:F/QMBIII
- added DEBUG: (no value), MICROCONTROLLER:6POS_JST
- added ENDSTOP, FAN, LIGHT: (no value), MICROCONTROLLER:2POS_JSTVERT_2.00
- added R13: (no value), MICROCONTROLLER:CAPC1005X35N
- added SPKR: F/QMBIII, buzzer:F/QMBIII
- added U$1: (no value), MICROCONTROLLER:LOGO_B
- moved PD0 2.00 mm to (53.8, 46.7)
- moved PD1 2.00 mm to (51.2, 46.7)
- moved PD2 2.00 mm to (48.8, 46.7)
- moved PE5 2.00 mm to (56.3, 46.7)
- moved J2 1.50 mm to (65.2, 55.7)
- moved C1 0.50 mm to (49.0, 63.6)
- moved C10 0.50 mm to (38.3, 42.7)
- moved C11 0.50 mm to (36.6, 44.6)
- moved C12 0.50 mm to (35.6, 44.6)
- moved C13 0.50 mm to (32.2, 39.2)
- moved C14 0.50 mm to (33.9, 38.0)
- moved C15 0.50 mm to (37.0, 38.0)
- moved C16 0.50 mm to (38.2, 39.3)
- moved C17 0.50 mm to (18.5, 9.25)
- moved C2 0.50 mm to (36.1, 76.4)
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Connections:
- new net N$15: ENDSTOP.1, R13.1, U1.59
- net +3V3: now also LIGHT.1, R13.2; no longer J3.1
- net +5V: now also FAN.1, SPKR.+; no longer J4.1, SG1.+
- net FAN_OUT: now also FAN.2; no longer J4.2
- net GND: now also ENDSTOP.2
- net LT: now also LIGHT.2; no longer J3.2
- net N$2: now also SPKR.-; no longer SG1.-
- net RXD: now also DEBUG.6; no longer J7.6
- net TCK: now also DEBUG.4; no longer J7.4
- net TDI: now also DEBUG.2; no longer J7.2
- net TDO: now also DEBUG.1; no longer J7.1
- net TMS: now also DEBUG.3; no longer J7.3
- net TXD: now also DEBUG.5; no longer J7.5
Routing:
- net GND: track 51.7 -> 76.2 mm, vias 11 -> 17
- net N$15: track 0.00 -> 11.3 mm
- net VDDC: track 9.73 -> 17.7 mm
- net +3V3: track 238.0 -> 243.6 mm
- net +5V: track 91.8 -> 90.2 mm
- net N$3: track 9.81 -> 10.8 mm
- net N$4: track 11.5 -> 12.5 mm
- net PE5: track 17.7 -> 16.8 mm
- net RXD: track 44.0 -> 44.8 mm
- net RX-1: track 13.7 -> 12.9 mm
- net TX-0: track 16.5 -> 15.7 mm
- net TMS: track 24.6 -> 25.3 mm
- net TDO: track 23.8 -> 24.4 mm
- net TCK: track 25.0 -> 25.7 mm
- net TDI: track 24.2 -> 24.9 mm
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- added copper zone on layer 16, net GND
Other:
- board size 69.5 x 84.8 mm -> 70 x 85 mm
- board text added: "BRANDON IAMS EE 474 FINAL PROJECT"

Commit message: fixing...
Connections:
- net GND: now also U3.6

Commit message: merge :
Connections:
- net GND: no longer U3.6
